File: _autosave-macropad.kicad_pcb (KiCad board)
At the start: 2 copper layers, 74.5 x 75 mm, 6 parts, among them J1 OLED_128x32, SW1 SW_Push, SW2 SW_Push, SW3 SW_Push, SW4 RotaryEncoder_Switch, U1 MOUDLE-SEEEDUINO-XIAO

Commit message: changing to simple 3 keys wip
Parts:
- removed J1: OLED_128x32, XIAO_PCB:OLED_128x32
- removed SW4: RotaryEncoder_Switch, Rotary_Encoder:RotaryEncoder_Alps_EC11E-Switch_Vertical_H20mm
- moved SW2 19.3 mm to (142.5, 99.4)
- moved SW3 19.3 mm to (161.5, 99.4)
- moved SW1 19.3 mm to (123.5, 99.4)
- moved U1 13.2 mm to (140.9, 63.5)
Connections:
- SW3 pad 1: Net-(U1-PA11_A3_D3) -> Net-(U1-PA7_A8_D8_SCK)
- U1 pad 1: Net-(U1-PA02_A0_D0) -> unconnected-(U1-PA02_A0_D0-Pad1)
- U1 pad 4: Net-(U1-PA11_A3_D3) -> unconnected-(U1-PA11_A3_D3-Pad4)
- U1 pad 5: Net-(J1-SDA) -> unconnected-(U1-PA8_A4_D4_SDA-Pad5)
- U1 pad 6: Net-(J1-SCL) -> unconnected-(U1-PA9_A5_D5_SCL-Pad6)
- U1 pad 8: EC11A -> unconnected-(U1-PB09_A7_D7_RX-Pad8)
- U1 pad 9: EC11B -> Net-(U1-PA7_A8_D8_SCK)
Routing:
- net EC11A: track 104.3 -> 0.00 mm
- net Net-(U1-PA02_A0_D0): track 82.5 -> 0.00 mm
- net EC11B: track 59.5 -> 0.00 mm
- net Net-(U1-PA11_A3_D3): track 59.2 -> 0.00 mm
- net GND: track 136.7 -> 87.2 mm
- net Net-(U1-PA7_A8_D8_SCK): track 0.00 -> 37.2 mm
- net +3.3V: track 35.6 -> 0.00 mm
- net Net-(J1-SDA): track 23.5 -> 0.00 mm
- net Net-(J1-SCL): track 22.8 -> 0.00 mm
- net Net-(U1-PA5_A9_D9_MISO): track 52.0 -> 35.8 mm
- net Net-(U1-PA6_A10_D10_MOSI): track 62.4 -> 46.3 mm
Other:
- board size 74.5 x 75 mm -> 57 x 61 mm
